File: Flux.sch (KiCad schematic (older format))
At the start: 191 parts, among them Q1 2N7002, SW2 SW_Push, SW3 SW_SPDT, U2 PRTR5V0U2X, U3 STM32F072CBUx, U4 MCP1700-3002E_SOT23

Commit message: Progress
Parts:
- removed C1, C10, C11, C12, C13, C14, C15, C16, C17, C18, C5, C9: 0.1uF, Capacitors_SMD:C_0603, symbol Device:C_Small
- removed D1, D19, D20, D21, D22, D23, D24, D25, D26, D27, D34, D35, D36, D37, D38, D39, D40, D41, D42, D47, D48, D49, D50, D51, D52, D53, D54, D55, D58, D59, D60, D61, D62, D63, D64, D67: SOD-123, Diodes_SMD:D_SOD-123, symbol Device:D_Small
- removed K_,1, K_.1, K_;1, K_B1, K_C1, K_D1, K_E1, K_F1, K_G1, K_H1, K_I1, K_J1, K_K1, K_L1, K_M1, K_N1, K_O1, K_P1, K_R1, K_RSHIFT3, K_SPACE3, K_T1, K_U1, K_V1, K_WIN1, K_X1, K_Y1: MX-1U, MX_Alps_Hybrid:MX-1U, symbol MX_Alps_Hybrids:MX-1U
- removed K_ALT1, K_CTRL1, K_ENTER2, K_RALT1, K_RCTRL1, K_SHIFT2: MX-1.25U, MX_Alps_Hybrid:MX-1.25U, symbol MX_Alps_Hybrids:MX-1U
- removed K_CAPS2: MX-1.25U, MX_Alps_Hybrid:MX-1.25U-FLIPPED, symbol MX_Alps_Hybrids:MX-1U
- removed K_ENTER1: MX-2.25U, MX_Alps_Hybrid:MX-2.25U, symbol MX_Alps_Hybrids:MX-1U
- removed K_ENTER3: MX-ISO, MX_Alps_Hybrid:MX-ISO-ReversedStabilizers, symbol MX_Alps_Hybrids:MX-1U
- removed K_LSPACE1: MX-2.25U, MX_Alps_Hybrid:MX-2.25U-ReversedStabilizers, symbol MX_Alps_Hybrids:MX-1U
- removed K_LSPACE2: MX-2.75U, MX_Alps_Hybrid:MX-2.75U-FLIPPED-ReversedStabilizers, symbol MX_Alps_Hybrids:MX-1U
- removed K_RSHIFT1, K_RSHIFT2: MX-1.75U, MX_Alps_Hybrid:MX-1.75U, symbol MX_Alps_Hybrids:MX-1U
- removed K_RSHIFT4: MX-2.75U, MX_Alps_Hybrid:MX-2.75U, symbol MX_Alps_Hybrids:MX-1U
- removed K_RSPACE1: MX-2.75U, MX_Alps_Hybrid:MX-2.75U-ReversedStabilizers, symbol MX_Alps_Hybrids:MX-1U
- removed K_RSPACE2: MX-2.25U, MX_Alps_Hybrid:MX-2.25U-FLIPPED-ReversedStabilizers, symbol MX_Alps_Hybrids:MX-1U
- removed K_RWIN1: MX-1.25U, MX_Alps_Hybrid:MX-1U, symbol MX_Alps_Hybrids:MX-1U
- removed K_SPACE2: MX-6U, MX_Alps_Hybrid:MX-6U-ReversedStabilizers, symbol MX_Alps_Hybrids:MX-1U
- removed K_SPACE4: MX-1U, MX_Alps_Hybrid:MX-1U-FLIPPED, symbol MX_Alps_Hybrids:MX-1U
- removed K_\1: MX-1.5U, MX_Alps_Hybrid:MX-1.5U, symbol MX_Alps_Hybrids:MX-1U
- removed Q1: 2N7002, TO_SOT_Packages_SMD:SOT-23, symbol Transistor_FET:2N7002
- removed R1, R16, R17, R18, R19, R20, R21, R22, R23, R24, R25, R26, R27, R31, R32, R33, R34, R35, R36, R37, R38, R39, R40, R41, R42, R44, R45, R46, R47, R48, R49, R50, R51, R52, R53, R54, R55, R58, R59, R60, R61, R62, R63, R64, R72: 1k, Resistors_SMD:R_0805, symbol Device:R_Small
- removed R3: 5.1k, Resistors_SMD:R_0805, symbol Device:R_Small
- removed R69: 100, Resistors_SMD:R_0805, symbol Device:R_Small
- removed RGB1, RGB10, RGB11, RGB12, RGB2, RGB3, RGB4, RGB5, RGB6, RGB7, RGB8, RGB9: WS2812B, LEDs:LED_WS2812B-PLCC4, symbol LED:WS2812B
- added C?: 1uF, symbol Device:C_Small
- added C? (x2): 0.1uF, symbol Device:C_Small
- added R?: 10k, symbol Device:R_Small
- added R?: 20k, symbol Device:R_Small
- added U?: IS31FL3731-QFLS2, symbol random-keyboard-parts:IS31FL3731-QFLS2
- renumbered D16 to D?, D17 to D?, D18 to D?, D31 to D?, D32 to D?, D33 to D?, D45 to D?, D46 to D?, D44 to D?, K_TAB1 to MX?, K_Q1 to MX?, K_W1 to MX?, K_CAPS1 to MX?, K_A1 to MX?, K_S1 to MX?, K_SHIFT1 to MX?, K_Z1 to MX?, K_SHIFT3 to MX?
Connections:
- net labels added: SCL, SDA
- net labels removed: .-COL, .-LEDGND, .-ROW, LEDGND
- wire segments 534 -> 122
- no-connect marks 8 -> 5
Other:
- moved on the sheet: D?, MX?
