File: Aurora.sch (KiCad schematic (older format))
At the start: 51 parts, among them SW2 SW_Push, SW3 SW_SPDT, U1 IS31FL3731-QFLS2, U2 PRTR5V0U2X, U3 STM32F072CBUx, U4 MCP1700-3002E_SOT23

Commit message: Begin replace LED MCU
Parts:
- removed U1: IS31FL3731-QFLS2, Housings_DFN_QFN:QFN-28-1EP_4x4mm_Pitch0.4mm, symbol random-keyboard-parts:IS31FL3731-QFLS2
- added C3, C5, C7, C8: 0.47uF, Capacitors_SMD:C_0603, symbol Device:C_Small
- added C4, C6: 0.1uF, Capacitors_SMD:C_0603, symbol Device:C_Small
- added R5: 20k, Resistors_SMD:R_0805, symbol Device:R_Small
- added U1: IS31FL3736, Housings_DFN_QFN:QFN-40-1EP_5x5mm_Pitch0.4mm, symbol random-keyboard-parts:IS31FL3736
- C1: value 10uF -> 22uF; footprint Capacitors_Tantalum_SMD:CP_Tantalum_Case-A_EIA-3216-18_Reflow -> Capacitors_Tantalum_SMD:CP_Tantalum_Case-T_EIA-3528-12_Reflow
- R3, R4: value 2k -> 1k
Connections:
- net +3V3: now also C8.1, U1.31 (VIO)
- net +5V: now also C3.1, C4.1, C5.1, C6.1, C7.1, U1.17 (PVCC), U1.23 (PVCC), U1.27 (DVCC), U1.28 (AVCC), U1.38 (SDB)
- net GND: now also C3.2, C4.2, C5.2, C6.2, C7.2, C8.2, R5.1, U1.11 (PGND), U1.26 (AGND), U1.35 (ADDR1), U1.36 (ADDR2), U1.4 (PGND), U1.40 (GND), U1.41 (Thermal)
- net SCL: now also U1.34 (SCL)
- net SDA: now also U1.33 (SDA)
- net at R1.2: now also U1.39 (IICRST)
- removed net CB1: LED1.2 (C), LED2.2 (C), LED3.2 (C), LED4.2 (C), LED5.2 (C), LED9.1 (A), LED9.1 (A), LED9.1 (A)
- removed net CB2: LED1.3 (C), LED2.3 (C), LED3.3 (C), LED4.3 (C), LED5.3 (C), LED8.1 (A), LED8.1 (A), LED8.1 (A)
- removed net CB3: LED1.4 (C), LED2.4 (C), LED3.4 (C), LED4.4 (C), LED5.4 (C), LED7.1 (A), LED7.1 (A), LED7.1 (A)
- removed net CB4: LED6.1 (A), LED6.1 (A), LED6.1 (A)
- removed net CB5: LED5.1 (A), LED5.1 (A), LED5.1 (A)
- removed net CB6: LED4.1 (A), LED4.1 (A), LED4.1 (A)
- removed net CB7: LED3.1 (A), LED3.1 (A), LED3.1 (A), LED6.4 (C), LED7.4 (C), LED8.4 (C), LED9.4 (C)
- removed net CB8: LED2.1 (A), LED2.1 (A), LED2.1 (A), LED6.3 (C), LED7.3 (C), LED8.3 (C), LED9.3 (C)
- removed net CB9: LED1.1 (A), LED1.1 (A), LED1.1 (A), LED6.2 (C), LED7.2 (C), LED8.2 (C), LED9.2 (C)
- new net: R5.2, U1.30 (RSET)
- new net CS1: U1.15 (CS1)
- new net CS2: U1.16 (CS2)
- new net CS3: U1.18 (CS3)
- new net CS4: U1.19 (CS4)
- new net CS5: U1.21 (CS5)
- new net CS6: U1.22 (CS6)
- new net CS7: U1.24 (CS7)
- new net CS8: U1.25 (CS8)
- new net SW1: U1.1 (SW1)
- new net SW10: U1.12 (SW10)
- new net SW11: U1.13 (SW11)
- new net SW12: U1.14 (SW12)
- new net SW2: U1.2 (SW2)
- new net SW3: U1.3 (SW3)
- new net SW4: U1.5 (SW4)
- new net SW5: U1.6 (SW5)
- new net SW6: U1.7 (SW6)
- new net SW7: U1.8 (SW7)
- new net SW8: U1.9 (SW8)
- new net SW9: U1.10 (SW9)
- no-connect marks 5 -> 7
Other:
- moved on the sheet: R3, R4

Commit message: Route it
Parts:
- D1, D2, D3, D4, D5, D6, D7, D8, D9: footprint Diodes_SMD:D_SOD-123 -> Diodes_SMD:D_SOD-323
- R1, R2, R3, R4, R5, R73, R74: footprint Resistors_SMD:R_0805 -> Resistors_SMD:R_0603
Connections:
- net CS1: now also LED1.1 (A), LED1.1 (A), LED1.1 (A), LED9.1 (A), LED9.1 (A), LED9.1 (A)
- net CS2: now also LED2.1 (A), LED2.1 (A), LED2.1 (A)
- net CS3: now also LED3.1 (A), LED3.1 (A), LED3.1 (A)
- net CS4: now also LED4.1 (A), LED4.1 (A), LED4.1 (A)
- net CS5: now also LED5.1 (A), LED5.1 (A), LED5.1 (A)
- net CS6: now also LED6.1 (A), LED6.1 (A), LED6.1 (A)
- net CS7: now also LED7.1 (A), LED7.1 (A), LED7.1 (A)
- net CS8: now also LED8.1 (A), LED8.1 (A), LED8.1 (A)
- net SW1: now also LED1.3 (C), LED2.3 (C), LED3.3 (C), LED4.3 (C), LED5.3 (C), LED6.3 (C), LED7.3 (C), LED8.3 (C)
- net SW2: now also LED1.2 (C), LED2.2 (C), LED3.2 (C), LED4.2 (C), LED5.2 (C), LED6.2 (C), LED7.2 (C), LED8.2 (C)
- net SW3: now also LED1.4 (C), LED2.4 (C), LED3.4 (C), LED4.4 (C), LED5.4 (C), LED6.4 (C), LED7.4 (C), LED8.4 (C)
- net SW4: now also LED9.3 (C)
- net SW5: now also LED9.2 (C)
- net SW6: now also LED9.4 (C)
Other:
- moved on the sheet: LED1A, LED1B, LED1C, LED2A, LED2B, LED2C, LED3A, LED3B, LED3C, LED4A, LED4B, LED4C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
