File: Aurora.kicad_pcb (KiCad board)
At the start: 2 copper layers, 57.1 x 62.7 mm, 51 parts, among them SW2 SW_Push, SW3 SW_SPDT, U1 IS31FL3731-QFLS2, U2 PRTR5V0U2X, U3 STM32F072CBUx, U4 MCP1700-3002E_SOT23

Commit message: Begin replace LED MCU
Parts:
- added C3: 0.47uF, Capacitors_SMD:C_0603, B.Cu at (75.4, 67.5)
- added C4: 0.1uF, Capacitors_SMD:C_0603, B.Cu at (66.7, 59.5)
- added C5: 0.47uF, Capacitors_SMD:C_0603, B.Cu at (66.7, 57.9)
- added C6: 0.1uF, Capacitors_SMD:C_0603, B.Cu at (68.3, 70.6)
- added C7: 0.47uF, Capacitors_SMD:C_0603, B.Cu at (68.3, 72.2)
- added C8: 0.47uF, Capacitors_SMD:C_0603, B.Cu at (74.6, 69.8)
- added R5: 20k, Resistors_SMD:R_0805, B.Cu at (72.2, 50.0)
- C1: value 10uF -> 22uF; footprint Capacitors_Tantalum_SMD:CP_Tantalum_Case-A_EIA-3216-18_Reflow -> Capacitors_Tantalum_SMD:CP_Tantalum_Case-T_EIA-3528-12_Reflow
- R3, R4: value 2k -> 1k
- U1: value IS31FL3731-QFLS2 -> IS31FL3736; footprint Housings_DFN_QFN:QFN-28-1EP_4x4mm_Pitch0.4mm -> Housings_DFN_QFN:QFN-40-1EP_5x5mm_Pitch0.4mm
- moved C1 10.3 mm to (80.2, 68.3), turned to 0 degrees
- moved R1 9.05 mm to (71.4, 80.2), turned to 0 degrees
- moved C2 4.27 mm to (73.8, 67.5), turned to 90 degrees
- moved U1 3.60 mm to (68.2, 65.1), turned to 0 degrees
- moved C24 0.79 mm to (57.1, 69.1)
Connections:
- net CA1 renamed CS5
- net CA2 renamed CS6
- net CA4 renamed CS7
- net CA5 renamed CS8
- net CA9 renamed SW1
- net Net-(U1-Pad16) renamed CS2
- LED1 pad 1: CB9 -> Net-(LED1-Pad1)
- LED1 pad 2: CB1 -> Net-(LED1-Pad2)
- LED1 pad 3: CB2 -> Net-(LED1-Pad3)
- LED1 pad 4: CB3 -> Net-(LED1-Pad4)
- LED2 pad 1: CB8 -> Net-(LED2-Pad1)
- LED2 pad 2: CB1 -> Net-(LED2-Pad2)
- LED2 pad 3: CB2 -> Net-(LED2-Pad3)
- LED2 pad 4: CB3 -> Net-(LED2-Pad4)
- LED3 pad 1: CB7 -> Net-(LED3-Pad1)
- LED3 pad 2: CB1 -> Net-(LED3-Pad2)
- LED3 pad 3: CB2 -> Net-(LED3-Pad3)
- LED3 pad 4: CB3 -> Net-(LED3-Pad4)
- LED4 pad 1: CB6 -> Net-(LED4-Pad1)
- LED4 pad 2: CB1 -> Net-(LED4-Pad2)
- LED4 pad 3: CB2 -> Net-(LED4-Pad3)
- LED4 pad 4: CB3 -> Net-(LED4-Pad4)
- LED5 pad 1: CB5 -> Net-(LED5-Pad1)
- LED5 pad 2: CB1 -> Net-(LED5-Pad2)
- LED5 pad 3: CB2 -> Net-(LED5-Pad3)
- LED5 pad 4: CB3 -> Net-(LED5-Pad4)
- LED6 pad 1: CB4 -> Net-(LED6-Pad1)
- LED6 pad 2: CB9 -> Net-(LED6-Pad2)
- LED6 pad 3: CB8 -> Net-(LED6-Pad3)
- LED6 pad 4: CB7 -> Net-(LED6-Pad4)
- LED7 pad 1: CB3 -> Net-(LED7-Pad1)
- LED7 pad 2: CB9 -> Net-(LED7-Pad2)
- LED7 pad 3: CB8 -> Net-(LED7-Pad3)
- LED7 pad 4: CB7 -> Net-(LED7-Pad4)
- LED8 pad 1: CB2 -> Net-(LED8-Pad1)
- LED8 pad 2: CB9 -> Net-(LED8-Pad2)
- LED8 pad 3: CB8 -> Net-(LED8-Pad3)
- LED8 pad 4: CB7 -> Net-(LED8-Pad4)
- LED9 pad 1: CB1 -> Net-(LED9-Pad1)
- LED9 pad 2: CB9 -> Net-(LED9-Pad2)
- LED9 pad 3: CB8 -> Net-(LED9-Pad3)
- LED9 pad 4: CB7 -> Net-(LED9-Pad4)
- U1 pad 10: CB4 -> SW9
- U1 pad 11: CB5 -> GND
- U1 pad 12: CB6 -> SW10
- U1 pad 13: CB7 -> SW11
- U1 pad 14: CB8 -> SW12
- U1 pad 15: CB9 -> CS1
- U1 pad 17: Net-(U1-Pad17) -> +5V
- U1 pad 18: GND -> CS3
- U1 pad 19: SDA -> CS4
- U1 pad 2: +5V -> SW2
- U1 pad 20: SCL -> (no net)
- U1 pad 23: CA3 -> +5V
- U1 pad 26: CA6 -> GND
- U1 pad 27: CA7 -> +5V
- U1 pad 28: CA8 -> +5V
- U1 pad 29: GND -> (no net)
- U1 pad 3: +5V -> SW3
- U1 pad 4: Net-(U1-Pad4) -> GND
- U1 pad 5: GND -> SW4
- U1 pad 6: Net-(R1-Pad2) -> SW5
- U1 pad 7: CB1 -> SW6
- U1 pad 8: CB2 -> SW7
- U1 pad 9: CB3 -> SW8
Routing:
- net GND: track 235.1 -> 52.8 mm, vias 9 -> 0
- net CB1: track 148.8 -> 0.00 mm, vias 6 -> 0
- net CB9: track 143.2 -> 0.00 mm, vias 8 -> 0
- net CB3: track 137.7 -> 0.00 mm, vias 8 -> 0
- net CB2: track 135.0 -> 0.00 mm, vias 7 -> 0
- net ROW0: track 116.4 -> 0.00 mm, vias 8 -> 0
- net CB7: track 113.7 -> 0.00 mm, vias 4 -> 0
- net CB8: track 108.5 -> 0.00 mm, vias 6 -> 0
- net ROW1: track 103.2 -> 0.00 mm, vias 6 -> 0
- net ROW2: track 101.2 -> 0.00 mm, vias 7 -> 0
- net COL2: track 92.1 -> 0.00 mm, vias 6 -> 0
- net +5V: track 99.6 -> 8.59 mm, vias 4 -> 0
- net +3V3: track 119.2 -> 44.0 mm, vias 13 -> 2
- net COL0: track 68.4 -> 0.00 mm, vias 5 -> 0
- net COL1: track 54.6 -> 0.00 mm, vias 4 -> 0
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Other:
- net class Default: clearance 0.2032 -> 0.1778; trace_width 0.254 -> 0.2032
- net class Power: clearance 0.2032 -> 0.1778
- rule trace_clearance: 0.2032 -> 0.1778

Commit message: Route it
Parts:
- D1, D2, D3, D4, D5, D6, D7, D8, D9: footprint Diodes_SMD:D_SOD-123 -> Diodes_SMD:D_SOD-323
- R1, R2, R3, R4, R5, R73, R74: footprint Resistors_SMD:R_0805 -> Resistors_SMD:R_0603
- moved R1 4.74 mm to (66.8, 79.5), turned to 180 degrees
- moved R4 2.29 mm to (65.9, 76.4), turned to 270 degrees
- moved R3 0.92 mm to (67.6, 76.4), turned to 270 degrees
- moved R74 0.85 mm to (52.7, 42.2)
- moved D6 0.30 mm to (65.4, 82.5)
- moved D7 0.30 mm to (84.4, 44.5)
- moved D8 0.30 mm to (84.4, 63.5)
- moved D9 0.30 mm to (84.4, 82.5)
- moved C6 0.29 mm to (68.3, 70.4)
- moved C7 0.22 mm to (68.3, 72.0)
Connections:
- LED1 pad 1: Net-(LED1-Pad1) -> CS1
- LED1 pad 2: Net-(LED1-Pad2) -> SW2
- LED1 pad 3: Net-(LED1-Pad3) -> SW1
- LED1 pad 4: Net-(LED1-Pad4) -> SW3
- LED2 pad 1: Net-(LED2-Pad1) -> CS2
- LED2 pad 2: Net-(LED2-Pad2) -> SW2
- LED2 pad 3: Net-(LED2-Pad3) -> SW1
- LED2 pad 4: Net-(LED2-Pad4) -> SW3
- LED3 pad 1: Net-(LED3-Pad1) -> CS3
- LED3 pad 2: Net-(LED3-Pad2) -> SW2
- LED3 pad 3: Net-(LED3-Pad3) -> SW1
- LED3 pad 4: Net-(LED3-Pad4) -> SW3
- LED4 pad 1: Net-(LED4-Pad1) -> CS4
- LED4 pad 2: Net-(LED4-Pad2) -> SW2
- LED4 pad 3: Net-(LED4-Pad3) -> SW1
- LED4 pad 4: Net-(LED4-Pad4) -> SW3
- LED5 pad 1: Net-(LED5-Pad1) -> CS5
- LED5 pad 2: Net-(LED5-Pad2) -> SW2
- LED5 pad 3: Net-(LED5-Pad3) -> SW1
- LED5 pad 4: Net-(LED5-Pad4) -> SW3
- LED6 pad 1: Net-(LED6-Pad1) -> CS6
- LED6 pad 2: Net-(LED6-Pad2) -> SW2
- LED6 pad 3: Net-(LED6-Pad3) -> SW1
- LED6 pad 4: Net-(LED6-Pad4) -> SW3
- LED7 pad 1: Net-(LED7-Pad1) -> CS7
- LED7 pad 2: Net-(LED7-Pad2) -> SW2
- LED7 pad 3: Net-(LED7-Pad3) -> SW1
- LED7 pad 4: Net-(LED7-Pad4) -> SW3
- LED8 pad 1: Net-(LED8-Pad1) -> CS8
- LED8 pad 2: Net-(LED8-Pad2) -> SW2
- LED8 pad 3: Net-(LED8-Pad3) -> SW1
- LED8 pad 4: Net-(LED8-Pad4) -> SW3
- LED9 pad 1: Net-(LED9-Pad1) -> CS1
- LED9 pad 2: Net-(LED9-Pad2) -> SW5
- LED9 pad 3: Net-(LED9-Pad3) -> SW4
- LED9 pad 4: Net-(LED9-Pad4) -> SW6
Routing:
- net GND: track 52.8 -> 335.0 mm, vias 0 -> 15
- net SW1: track 0.00 -> 192.6 mm, vias 0 -> 10
- net SW2: track 0.00 -> 189.3 mm, vias 0 -> 14
- net SW3: track 0.00 -> 167.9 mm, vias 0 -> 9
- net +3V3: track 44.0 -> 181.0 mm, vias 2 -> 11
- net +5V: track 8.59 -> 118.6 mm, vias 0 -> 8
- net COL2: track 0.00 -> 99.9 mm, vias 0 -> 7
- net ROW1: track 0.00 -> 95.6 mm, vias 0 -> 5
- net ROW2: track 0.00 -> 88.7 mm, vias 0 -> 4
- net ROW0: track 0.00 -> 71.1 mm, vias 0 -> 3
- net CS1: track 0.00 -> 69.0 mm, vias 0 -> 5
- net COL0: track 0.00 -> 68.6 mm, vias 0 -> 7
- net COL1: track 0.00 -> 64.7 mm, vias 0 -> 6
- net CS7: track 0.00 -> 49.9 mm, vias 0 -> 4
- net CS4: track 0.00 -> 40.8 mm, vias 0 -> 4
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
Commit message: Route PCB
Parts:
- added G***: LOGO, locallib:ai-ring-6mm, F.Cu at (73.2, 68.4)
- moved F1 0.51 mm to (45.6, 48.8)
Routing:
- net +3V3: track 181.0 -> 163.9 mm
- net Net-(R74-Pad2): track 17.2 -> 11.8 mm
- net SW2: track 189.3 -> 192.6 mm, vias 14 -> 12
- net SW1: track 192.6 -> 189.6 mm
- net VCC: track 24.6 -> 27.5 mm, vias 2 -> 4
- net GND: track 335.0 -> 337.7 mm
- net COL0: track 68.6 -> 66.5 mm
- net SWDIO: track 2.07 -> 0.00 mm
- net CS1: track 69.0 -> 67.1 mm, vias 5 -> 3
- net SW4: track 30.1 -> 32.0 mm
- net CS2: track 29.9 -> 28.1 mm
- net SW3: track 167.9 -> 166.4 mm, vias 9 -> 8
- net CS3: track 31.6 -> 30.1 mm
- net +5V: track 118.6 -> 120.0 mm
- net COL2: track 99.9 -> 101.2 mm
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- added copper zone on B.Cu, net GND
Other:
- board text added: "AURORA"
- board text added: "Aurora PCB 1.0 by ai03"
