File: Aurora.kicad_pcb (KiCad board)
At the start: 2 copper layers, 57.1 x 62.7 mm, 59 parts, among them SW2 SW_Push, SW3 SW_SPDT, U1 IS31FL3736, U2 PRTR5V0U2X, U3 STM32F072CBUx, U4 MCP1700-3002E_SOT23

Commit message: Further tuning
Routing:
- net VCC: track 27.5 -> 26.2 mm
- net GND: track 337.7 -> 337.1 mm
Changed lines of the file:
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@@
     (thickness 1.6)
     (drawings 21)
-    (tracks 1517)
+    (tracks 1516)
     (zones 0)
     (modules 59)
@@
   (segment (start 52.705 42.914) (end 52.4644 42.914) (width 0.381) (layer B.Cu) (net 2))
   (segment (start 50.2125 40.6621) (end 50.2125 40.525) (width 0.381) (layer B.Cu) (net 2))
-  (segment (start 52.4644 42.914) (end 50.2125 40.6621) (width 0.381) (layer B.Cu) (net 2))
-  (segment (start 49.6824 40.8432) (end 49.3776 40.5384) (width 0.381) (layer F.Cu) (net 2))
   (via (at 47.1424 40.3352) (size 0.6) (drill 0.4) (layers F.Cu B.Cu) (net 2))
-  (segment (start 49.3776 40.5384) (end 49.1744 40.3352) (width 0.381) (layer F.Cu) (net 2))
-  (segment (start 49.1744 40.3352) (end 47.1424 40.3352) (width 0.381) (layer F.Cu) (net 2))
   (segment (start 46.9392 40.5384) (end 47.1424 40.3352) (width 0.381) (layer B.Cu) (net 2))
   (segment (start 46.6344 40.8432) (end 46.9392 40.5384) (width 0.381) (layer B.Cu) (net 2))
@@
   (segment (start 52.705 42.914) (end 51.4484 42.914) (width 0.381) (layer B.Cu) (net 2))
   (segment (start 51.4484 42.914) (end 51.4096 42.8752) (width 0.381) (layer B.Cu) (net 2))
-  (segment (start 51.4096 42.8752) (end 51.4096 42.5704) (width 0.381) (layer F.Cu) (net 2))
-  (segment (start 49.6824 40.8432) (end 51.4096 42.5704) (width 0.381) (layer F.Cu) (net 2))
   (segment (start 49.5808 73.66) (end 49.5808 75.4888) (width 0.381) (layer B.Cu) (net 2))
   (segment (start 47.8536 71.3232) (end 45.5168 68.9864) (width 0.381) (layer F.Cu) (net 2))
@@
   (segment (start 65.4304 39.116) (end 65.4304 42.4688) (width 0.381) (layer F.Cu) (net 2))
   (segment (start 65.4304 42.4688) (end 65.4304 43.688) (width 0.381) (layer F.Cu) (net 2))
+  (segment (start 51.4096 41.8592) (end 51.2064 41.656) (width 0.381) (layer B.Cu) (net 2))
+  (segment (start 51.4096 42.8752) (end 51.4096 41.8592) (width 0.381) (layer B.Cu) (net 2))
+  (segment (start 51.2064 41.656) (end 50.2125 40.6621) (width 0.381) (layer B.Cu) (net 2))
+  (segment (start 48.8696 40.3352) (end 49.276 40.7416) (width 0.381) (layer F.Cu) (net 2))
+  (segment (start 47.1424 40.3352) (end 48.8696 40.3352) (width 0.381) (layer F.Cu) (net 2))
+  (segment (start 51.4096 42.8752) (end 49.276 40.7416) (width 0.381) (layer F.Cu) (net 2))
   (segment (start 45.5295 34.6075) (end 45.4533 34.6075) (width 0.2032) (layer B.Cu) (net 3))
   (segment (start 45.4533 34.6075) (end 42.8752 37.1856) (width 0.2032) (layer B.Cu) (net 3))
@@
   (segment (start 48.2125 40.5859) (end 48.2125 40.325) (width 0.381) (layer B.Cu) (net 7))
   (segment (start 47.244 41.5544) (end 48.2125 40.5859) (width 0.381) (layer B.Cu) (net 7))
-  (via (at 43.8912 47.752) (size 0.6) (drill 0.4) (layers F.Cu B.Cu) (net 7))
-  (segment (start 45.6184 47.568) (end 44.0752 47.568) (width 0.381) (layer B.Cu) (net 7))
-  (segment (start 44.0752 47.568) (end 43.8912 47.752) (width 0.381) (layer B.Cu) (net 7))
   (segment (start 47.244 41.5544) (end 47.244 43.2816) (width 0.381) (layer B.Cu) (net 7))
-  (via (at 46.3296 44.3992) (size 0.6) (drill 0.4) (layers F.Cu B.Cu) (net 7))
-  (segment (start 47.244 43.2816) (end 46.3296 44.196) (width 0.381) (layer B.Cu) (net 7))
-  (segment (start 46.3296 44.196) (end 46.3296 44.3992) (width 0.381) (layer B.Cu) (net 7))
-  (segment (start 46.3296 45.3136) (end 43.8912 47.752) (width 0.381) (layer F.Cu) (net 7))
-  (segment (start 46.3296 44.3992) (end 46.3296 45.3136) (width 0.381) (layer F.Cu) (net 7))
+  (via (at 47.244 44.3992) (size 0.6) (drill 0.4) (layers F.Cu B.Cu) (net 7))
+  (segment (start 47.244 43.2816) (end 47.244 44.3992) (width 0.381) (layer B.Cu) (net 7))
+  (via (at 47.4472 47.5488) (size 0.6) (drill 0.4) (layers F.Cu B.Cu) (net 7))
+  (segment (start 47.428 47.568) (end 45.6184 47.568) (width 0.381) (layer B.Cu) (net 7))
+  (segment (start 47.4472 47.5488) (end 47.428 47.568) (width 0.381) (layer B.Cu) (net 7))
+  (segment (start 47.0408 47.1424) (end 47.4472 47.5488) (width 0.381) (layer F.Cu) (net 7))
+  (segment (start 47.244 44.3992) (end 47.0408 44.6024) (width 0.381) (layer F.Cu) (net 7))
+  (segment (start 47.0408 44.6024) (end 47.0408 47.1424) (width 0.381) (layer F.Cu) (net 7))
   (segment (start 47.90625 61.11425) (end 47.90625 61.8375) (width 0.2032) (layer B.Cu) (net 8))
   (via (at 43.688 60.0456) (size 0.6) (drill 0.4) (layers F.Cu B.Cu) (net 8))
@@
   (segment (start 51.6128 37.1872) (end 51.6525 37.1475) (width 0.2032) (layer B.Cu) (net 8))
   (segment (start 51.6128 39.2176) (end 51.6128 37.1872) (width 0.2032) (layer B.Cu) (net 8))
-  (segment (start 47.3456 39.2176) (end 46.5328 40.0304) (width 0.2032) (layer F.Cu) (net 8))
-  (segment (start 51.6128 39.2176) (end 47.3456 39.2176) (width 0.2032) (layer F.Cu) (net 8))
-  (segment (start 49.9872 53.4416) (end 49.9872 55.9816) (width 0.2032) (layer F.Cu) (net 8))
-  (segment (start 46.5328 40.0304) (end 46.5328 43.5864) (width 0.2032) (layer F.Cu) (net 8))
-  (segment (start 46.5328 43.5864) (end 46.9392 43.9928) (width 0.2032) (layer F.Cu) (net 8))
-  (segment (start 46.9392 43.9928) (end 46.9392 50.3936) (width 0.2032) (layer F.Cu) (net 8))
-  (segment (start 46.9392 50.3936) (end 49.9872 53.4416) (width 0.2032) (layer F.Cu) (net 8))
   (via (at 49.5808 55.88) (size 0.6) (drill 0.4) (layers F.Cu B.Cu) (net 8))
   (segment (start 51.6525 56.1975) (end 49.8983 56.1975) (width 0.2032) (layer B.Cu) (net 8))
@@
   (segment (start 49.9872 55.9816) (end 45.72 60.2488) (width 0.2032) (layer F.Cu) (net 8))
   (segment (start 45.72 60.2488) (end 43.8912 60.2488) (width 0.2032) (layer F.Cu) (net 8))
+  (segment (start 49.9872 53.4416) (end 49.9872 55.9816) (width 0.2032) (layer F.Cu) (net 8))
+  (segment (start 46.5328 49.9872) (end 49.9872 53.4416) (width 0.2032) (layer F.Cu) (net 8))
+  (segment (start 46.5328 40.0304) (end 46.5328 49.9872) (width 0.2032) (layer F.Cu) (net 8))
+  (segment (start 47.3456 39.2176) (end 46.5328 40.0304) (width 0.2032) (layer F.Cu) (net 8))
+  (segment (start 51.6128 39.2176) (end 47.3456 39.2176) (width 0.2032) (layer F.Cu) (net 8))
   (via (at 70.7136 54.1528) (size 0.6) (drill 0.4) (layers F.Cu B.Cu) (net 9))
   (segment (start 70.7025 56.1975) (end 70.7025 54.1639) (width 0.2032) (layer B.Cu) (net 9))
@@
   (segment (start 84.328 65.532) (end 84.328 44.3992) (width 0.381) (layer F.Cu) (net 17))
   (segment (start 82.2198 42.291) (end 73.7362 42.291) (width 0.381) (layer F.Cu) (net 17))
-  (via (at 56.1848 51.2064) (size 0.6) (drill 0.4) (layers F.Cu B.Cu) (net 17))
-  (segment (start 55.1688 52.2224) (end 56.1848 51.2064) (width 0.381) (layer B.Cu) (net 17))
   (segment (start 54.4576 52.2224) (end 55.1688 52.2224) (width 0.381) (layer B.Cu) (net 17))
   (segment (start 54.4576 52.2224) (end 53.4416 52.2224) (width 0.381) (layer B.Cu) (net 17))
   (via (at 57.8104 51.2064) (size 0.6) (drill 0.4) (layers F.Cu B.Cu) (net 17))
-  (segment (start 56.5912 51.2064) (end 57.8104 51.2064) (width 0.381) (layer F.Cu) (net 17))
-  (segment (start 56.1848 51.2064) (end 56.5912 51.2064) (width 0.381) (layer F.Cu) (net 17))
   (segment (start 57.912 51.1048) (end 57.8104 51.2064) (width 0.381) (layer B.Cu) (net 17))
   (segment (start 60.0456 51.1048) (end 57.912 51.1048) (width 0.381) (layer B.Cu) (net 17))
@@
   (segment (start 49.4792 58.2168) (end 49.784 58.2168) (width 0.381) (layer B.Cu) (net 17))
   (segment (start 47.8536 56.5912) (end 49.4792 58.2168) (width 0.381) (layer B.Cu) (net 17))
+  (via (at 56.0832 51.816) (size 0.6) (drill 0.4) (layers F.Cu B.Cu) (net 17))
+  (segment (start 55.1688 52.2224) (end 55.6768 52.2224) (width 0.381) (layer B.Cu) (net 17))
+  (segment (start 55.6768 52.2224) (end 56.0832 51.816) (width 0.381) (layer B.Cu) (net 17))
+  (segment (start 56.6928 51.2064) (end 56.0832 51.816) (width 0.381) (layer F.Cu) (net 17))
+  (segment (start 57.8104 51.2064) (end 56.6928 51.2064) (width 0.381) (layer F.Cu) (net 17))
   (segment (start 46.1125 80.7) (end 52.3125 80.7) (width 0.2032) (layer B.Cu) (net 18))
   (segment (start 46.1125 80.7) (end 45.284 80.7) (width 0.2032) (layer B.Cu) (net 18))

Commit message: Update readme
Routing:
- net GND: track 337.1 -> 334.4 mm
- net CS1: track 67.5 -> 68.4 mm
